File: KiCad/HV servo drive v1/phase bridges.kicad_sch (KiCad schematic)
At the start: 108 parts, among them Q1 C3M0075120K, Q2 C3M0075120K, Q3 C3M0075120K, Q4 C3M0075120K, Q5 C3M0075120K, Q6 C3M0075120K, U10 2EDF9275FXUMA1, U11 2EDF9275FXUMA1, U12 AMC1306M25DWVR, U13 2EDF9275FXUMA1, U14 AMC1306M25DWVR, U15 AMC1306M25DWVR

Commit message: KiCad 8.0 update
Parts:
- renumbered C80 to C10, C68 to C37, C45 to C40, C37 to C45, C70 to C46, C46 to C47, C40 to C50, C71 to C51, C47 to C52, C51 to C53, C73 to C54, C50 to C55, C54 to C56, C10 to C57, C77 to C58, C78 to C59, C52 to C60, C53 to C61, C61 to C62, C55 to C63, C62 to C64, C74 to C65, C79 to C66, C81 to C67, C82 to C68, C83 to C69, C56 to C70, C57 to C71, C58 to C72, C59 to C73, C75 to C74, C76 to C75, C84 to C76, C85 to C77, C60 to C78, C63 to C79, C66 to C80, C86 to C81, C64 to C82, C69 to C83, C87 to C84, C65 to C85, C72 to C86, C88 to C87, C67 to C88, D17 to D16, D21 to D17, D16 to D18, D22 to D19, D23 to D20, D18 to D21, D20 to D22, D24 to D23, D19 to D24, L14 to L11, L8 to L12, L9 to L13, L11 to L14, L4 to L3, L3 to L4, L12 to L8, L13 to L9, Q3 to Q1, Q4 to Q2, Q5 to Q3, Q6 to Q4, Q1 to Q5, Q2 to Q6, R48 to R33, R53 to R34, R33 to R35, R68 to R36, R56 to R47, R34 to R48, R51 to R49, R57 to R50, R35 to R51, R54 to R52, R55 to R53, R58 to R54, R59 to R55, R36 to R56, R47 to R57, R60 to R58, R61 to R59, R49 to R60, R63 to R61, R50 to R63, R66 to R64, R64 to R66, R52 to R68, TP13 to TP10, TP16 to TP11, TP14 to TP13, TP17 to TP14, TP10 to TP16, TP9 to TP17, TP11 to TP9, U11 to U10, U13 to U11, U10 to U12, U14 to U13, U15 to U14, U12 to U15

Commit message: start rev 2 changes
fix component references, fix rj45 and dc-dc converter footprints, add RLC filters on all power connectors, add more mounting holes
Parts:
- added C108, C109, C110, C111, C112, C113, C118, C119, C120, C121, C122, C123, C124, C125, C126, C127, C128, C129: C, Capacitor_SMD:C_1210_3225Metric, symbol Device:C
- renumbered C10 to C38, C40 to C39, C45 to C40, C47 to C41, C50 to C42, C52 to C43, C53 to C44, C55 to C45, C56 to C46, C57 to C47, C60 to C48, C61 to C49, C62 to C50, C63 to C51, C64 to C52, C65 to C53, C70 to C54, C71 to C55, C72 to C56, C73 to C57, C74 to C58, C75 to C59, C78 to C60, C79 to C61, C80 to C62, C82 to C63, C83 to C64, C85 to C65, C86 to C66, C88 to C67, C37 to C68, C46 to C69, C51 to C70, C54 to C71, C58 to C72, C59 to C73, C66 to C74, C67 to C75, C68 to C76, C69 to C77, C76 to C78, C77 to C79, C81 to C80, C84 to C81, C87 to C82, D18 to D10, D19 to D11, D21 to D12, D22 to D13, D24 to D14, D17 to D15, D20 to D16, D23 to D17, D16 to D9, L14 to L10, L8 to L11, L9 to L12, L11 to L13, L2 to L5, L3 to L6, L4 to L7, L12 to L8, L13 to L9, Q1 to Q2, Q2 to Q3, Q5 to Q4, Q6 to Q5, Q3 to Q6, Q4 to Q7, R33 to R36, R35 to R37, R36 to R38, R48 to R39, R49 to R40, R51 to R41, R52 to R42, R53 to R43, R56 to R44, R57 to R45, R58 to R46, R60 to R47, R61 to R48, R63 to R49, R64 to R50, R68 to R51, R34 to R52, R47 to R53, R50 to R54, R54 to R55, R55 to R56, R59 to R57, R62 to R58, R66 to R59, TP12 to TP10, TP13 to TP11, TP15 to TP12, TP17 to TP13, TP11 to TP14, TP14 to TP15, TP9 to TP8, TP10 to TP9, U10 to U14, U12 to U15, U13 to U16, U15 to U17, U11 to U18, U14 to U19
Connections:
- net +VDC: now also C108.1, C109.1, C110.1, C111.1, C112.1, C113.1, C118.1, C119.1, C120.1, C121.1, C122.1, C123.1, C124.1, C125.1, C126.1, C127.1, C128.1, C129.1
- net -VDC: now also C108.2, C109.2, C110.2, C111.2, C112.2, C113.2, C118.2, C119.2, C120.2, C121.2, C122.2, C123.2, C124.2, C125.2, C126.2, C127.2, C128.2, C129.2
- net U renamed U_
- net V renamed V_
- net W renamed W_
Other:
- moved on the sheet: C66, C67, C82, R46, R47, R48, R49, R50, R51, R57, R58, R59

Commit message: update to rev 2.1
basically the same version as in the FOC youtube video, with some minor issues fixed
Parts:
- removed L10, L11, L12, L13, L5, L6, L7, L8, L9: 10uH, Inductor_SMD:L_0603_1608Metric, symbol Device:L
- added C133, C136, C137: 470pf, Capacitor_SMD:C_1206_3216Metric, symbol Device:C
- added D35, D36, D37: RS1MLW, footprints:D_SOD-123W, symbol Device:D
- added FB1, FB2, FB3, FB4, FB5, FB6, FB7, FB8, FB9: 120 ohm, Inductor_SMD:L_0603_1608Metric, symbol Device:FerriteBead_Small
- added R108, R109, R91: 10, Resistor_SMD:R_1206_3216Metric, symbol Device:R
- added R8, R89, R9: 1, Resistor_SMD:R_0805_2012Metric, symbol Device:R
- C108, C109, C110, C111, C112, C113, C118, C119, C120, C121, C122, C123, C124, C125, C126, C127, C128, C129: value C -> 47nf; Generic Allowed? (none) -> no; Manufacturer (none) -> KEMET; Part number (none) -> C1210C473KDRACTU
- C38, C39, C44, C45, C50, C51, C54, C55, C58, C59, C60, C61, C64, C65, C68, C71, C74, C75, C78, C79, C81: Generic Allowed? (none) -> yes; Manufacturer (none) -> YAGEO; Part number (none) -> CC0603ZRY5V9BB104
- C40, C41, C42, C43, C46, C47, C48, C49, C52, C53, C56, C57, C69, C70, C72, C73, C76, C77: Generic Allowed? (none) -> yes; Manufacturer (none) -> Murata Electronics; Part number (none) -> GRM21BR61H106KE43L
- C62, C63, C80: value 2.2 -> 1uf; Generic Allowed? (none) -> yes; Manufacturer (none) -> Samsung Electro-Mechanics; Part number (none) -> CL10A105KB8NNNC
- C66, C67, C82, TP10, TP11, TP12, TP13, TP14, TP15, TP16, TP8, TP9: now not fitted
- D10, D11, D12, D15, D16, D9: value D -> RS1MLW; footprint Diode_SMD:D_SMB -> footprints:D_SOD-123W; Generic Allowed? (none) -> yes; Manufacturer (none) -> Taiwan Semiconductor Corporation; Part number (none) -> RS1MLW
- D13, D14, D17: Generic Allowed? (none) -> yes; Manufacturer (none) -> Micro Commercial Co; Part number (none) -> BZT52C5V1-TP
- Q2, Q3, Q4, Q5, Q6, Q7: value C3M0075120K -> G3R30MT12K; Generic Allowed? (none) -> no; Manufacturer (none) -> GeneSiC Semiconductor; Part number (none) -> G3R30MT12K; now not fitted
- R36, R37, R38, R39, R52, R53: Generic Allowed? (none) -> yes; Manufacturer (none) -> YAGEO; Part number (none) -> RC0805FR-131RL
- R40, R41, R54: value 800 -> 820; Generic Allowed? (none) -> yes; Manufacturer (none) -> YAGEO; Part number (none) -> RC0805JR-07820RL
- R42, R43, R44, R45, R55, R56: Generic Allowed? (none) -> yes; Manufacturer (none) -> YAGEO; Part number (none) -> RT1206FRE0710RL
- R46, R47, R50, R51, R57, R59: value R -> 0; Generic Allowed? (none) -> yes; Manufacturer (none) -> YAGEO; Part number (none) -> RC0603JR-070RL
- R48, R49, R58: Generic Allowed? (none) -> yes, must be low inductance shunt; Manufacturer (none) -> Stackpole Electronics Inc; Part number (none) -> HCSM2818FT5L00
- U14, U15, U18: value 2EDF9275FXUMA1 -> 2EDF8275FXUMA1; Generic Allowed? (none) -> no; Manufacturer (none) -> Infineon Technologies; Part number (none) -> 2EDF8275FXUMA1
- U16, U17, U19: Generic Allowed? (none) -> no; Manufacturer (none) -> Texas Instruments; Part number (none) -> AMC1306M25DWVR
Connections:
- net -5V: now also FB3.1, FB6.1, FB9.1
- net -VDC: now also C133.2, C136.2, C137.2
- net GND3: now also FB2.1, FB5.1, FB8.1
- net at C46.1, C50.1, D9.1 (K)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: now also D35.2 (A)
- net at C63.2, C65.2, D14.2 (A)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: now also R91.1
- net at C62.2, C64.2, D13.2 (A)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: now also R108.1
- net at C72.1, C74.1, D15.1 (K)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: now also D36.2 (A)
- net at C48.1, C54.1, D10.1 (K)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: now also D37.2 (A)
- net at C80.2, C81.2, D17.2 (A)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: now also R109.1
- net at C76.2, C77.1, C78.2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: now also FB5.2
- net at C77.2, C79.2, U18.9 (GNDB): now also FB6.2
- net at C76.1, C78.1, U18.11 (VDDB): now also FB4.2
- net at C56.1, C60.1, U15.11 (VDDB): now also FB7.2
- net at C56.2, C57.1, C60.2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: now also FB8.2
- net at C52.2, C53.1, C58.2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: now also FB2.2
- net at C53.2, C59.2, U14.9 (GNDB): now also FB3.2
- net at C57.2, C61.2, U15.9 (GNDB): now also FB9.2
- net at C52.1, C58.1, U14.11 (VDDB): now also FB1.2
- net +15V renamed +15V_GATE
- net +15V_GATE: now also FB1.1, FB4.1, FB7.1
- new net: C136.1, R108.2
- new net: D36.1 (K), R9.1
- new net: C137.1, R109.2
- new net: D37.1 (K), R89.1
- new net: C133.1, R91.2
- new net: D35.1 (K), R8.1
- new net VBUS +15V: R8.2, R89.2, R9.2
Other:
- moved on the sheet: R46, R47, R48, R49, R50, R51, R57, R58, R59

Commit message: add reverse protection diodes to gate supply
Parts:
- added D38, D39, D40: BAT54SLT1G, Package_TO_SOT_SMD:SOT-23, symbol Device:D_Dual_Series_AKC
Connections:
- net at C46.1, C50.1, D35.2 (A)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: now also D38.2 (K)
- net at C46.2, C47.1, C50.2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: now also D38.3 (common)
- net at C48.2, C49.1, C54.2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: now also D40.3 (common)
- net at C47.2, C51.2, D11.2 (A)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: now also D38.1 (A)
- net at C72.1, C74.1, D15.1 (K)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: now also D39.2 (K)
- net at C72.2, C73.1, C74.2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: now also D39.3 (common)
- net at C48.1, C54.1, D10.1 (K)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: now also D40.2 (K)
- net at C49.2, C55.2, D12.2 (A)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: now also D40.1 (A)
- net at C73.2, C75.2, D16.2 (A)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: now also D39.1 (A)
Other:
- moved on the sheet: C46, C47, C48, C49, C50, C51, C54, C55, C72, C73, C74, C75
